Commit message: Added the vgc10 gripper, and created the webots urdf

File: vgc10_description/urdf/ur.ros2_control.xacro (robot description, xacro)
@@ -22,5 +22,5 @@
           <param name="headless_mode">0</param>
           <param name="reverse_port">50001</param>
-          <param name="script_sender_port">50002</param>
+          <param name="script_sender_port">29999</param>
           <param name="tf_prefix">"${tf_prefix}"</param>
           <param name="non_blocking_read">0</param>

File: vgc10_description/urdf/ur_vgc10.urdf.xacro (robot description, xacro)
@@ -4,5 +4,5 @@
    <xacro:arg name="name" default="ur"/>
    <!-- import main macro -->
-   <xacro:include filename="$(find ur_description)/urdf/ur_macro.xacro"/>
+   <xacro:include filename="$(find vgc10_description)/urdf/ur_macro.xacro"/>
   <xacro:macro name="onrobot_vgc10_base_link" params="prefix">
     <link name="${prefix}onrobot_vgc10_base_link">
@@ -15,5 +15,5 @@
         <origin xyz="0 0 0" rpy="0 0 0" />
         <geometry>
-          <mesh filename="package://ur_description/meshes/visual/base_link.stl" />
+          <mesh filename="package://vgc10_description/meshes/visual/base_link.stl" />
         </geometry>
         <material name="">
@@ -24,5 +24,5 @@
         <origin xyz="0 0 0" rpy="0 0 0" />
         <geometry>
-          <mesh filename="package://ur_description/meshes/collision/base_link.stl" />
+          <mesh filename="package://vgc10_description/meshes/collision/base_link.stl" />
         </geometry>
       </collision>
@@ -49,5 +49,5 @@
         <origin xyz="0 0 0" rpy="0 0 0" />
         <geometry>
-          <mesh filename="package://ur_description/meshes/visual/suction_cup.stl" />
+          <mesh filename="package://vgc10_description/meshes/visual/suction_cup.stl" />
         </geometry>
         <material name="">
@@ -58,5 +58,5 @@
         <origin xyz="0 0 0" rpy="0 0 0" />
         <geometry>
-          <mesh filename="package://ur_description/meshes/collision/suction_cup.stl" />
+          <mesh filename="package://vgc10_description/meshes/collision/suction_cup.stl" />
         </geometry>
       </collision>
@@ -90,5 +90,5 @@
    <xacro:arg name="fake_sensor_commands" default="false" />
    <!-- initial position -->
-   <xacro:arg name="initial_positions_file" default="$(find ur_description)/config/initial_positions.yaml"/>
+   <xacro:arg name="initial_positions_file" default="$(find vgc10_description)/config/initial_positions.yaml"/>
    <xacro:property name="initial_positions_file" default="$(arg initial_positions_file)"/>
    <!-- arm -->

File: vgc10_description/urdf/ur_webots.urdf.xacro (robot description, xacro)
@@ -1,45 +1,96 @@
 <?xml version="1.0"?>
-<robot xmlns:xacro="http://wiki.ros.org/xacro">
-  <!--
-    Base UR robot series xacro macro.
-    NOTE this is NOT a URDF. It cannot directly be loaded by consumers
-    expecting a flattened '.urdf' file. See the top-level '.xacro' for that
-    (but note that .xacro must still be processed by the xacro command).
-    This file models the base kinematic chain of a UR robot, which then gets
-    parameterised by various configuration files to convert it into a UR3(e),
-    UR5(e), UR10(e) or UR16e.
-    NOTE the default kinematic parameters (i.e., link lengths, frame locations,
-    offsets, etc) do not correspond to any particular robot. They are defaults
-    only. There WILL be non-zero offsets between the Forward Kinematics results
-    in TF (i.e., robot_state_publisher) and the values reported by the Teach
-    Pendant.
-    For accurate (and robot-specific) transforms, the 'kinematics_parameters_file'
-    parameter MUST point to a .yaml file containing the appropriate values for
-    the targeted robot.
-    If using the UniversalRobots/Universal_Robots_ROS_Driver, follow the steps
-    described in the readme of that repository to extract the kinematic
-    calibration from the controller and generate the required .yaml file.
-    Main author of the migration to yaml configs Ludovic Delval.
-    Contributors to previous versions (in no particular order)
-     - Denis Stogl
-     - Lovro Ivanov
-     - Felix Messmer
-     - Kelsey Hawkins
-     - Wim Meeussen
-     - Shaun Edwards
-     - Nadia Hammoudeh Garcia
-     - Dave Hershberger
-     - G. vd. Hoorn
-     - Philip Long
-     - Dave Coleman
-     - Miguel Prada
-     - Mathias Luedtke
-     - Marcel Schnirring
-     - Felix von Drigalski
-     - Felix Exner
-     - Jimmy Da Silva
-     - Ajit Krisshna N L
-     - Muhammad Asif Rana
-  -->
+<robot xmlns:xacro="http://wiki.ros.org/xacro" name="$(arg name)">
+   <!-- robot name parameter -->
+   <xacro:arg name="name" default="ur"/>
+   <!-- import main macro -->
+  <webots>
+      <plugin type="webots_ros2_control::Ros2Control" />
+  </webots>
+  <xacro:macro name="onrobot_vgc10_base_link" params="prefix">
+    <link name="${prefix}onrobot_vgc10_base_link">
+      <inertial>
+        <origin xyz="0.0 0.0 0.0" rpy="0 0 0" />
+        <mass value="0.6" />
+        <inertia ixx="1.0E-03" ixy="1.0E-06" ixz="1.0E-06" iyy="1.0E-03" iyz="1.0E-06" izz="1.0E-03" />
+      </inertial>
+      <visual>
+        <origin xyz="0 0 0" rpy="0 0 0" />
+        <geometry>
+          <mesh filename="package://vgc10_description/meshes/visual/base_link.stl" />
+        </geometry>
+        <material name="">
+          <color rgba="0.8 0.8 0.8 1" />
+        </material>
+      </visual>
+      <collision>
+        <origin xyz="0 0 0" rpy="0 0 0" />
+        <geometry>
+          <mesh filename="package://vgc10_description/meshes/collision/base_link.stl" />
+        </geometry>
+      </collision>
+    </link>
+    <joint name="${prefix}onrobot_vgc10_joint" type="fixed">
+      <!-- The parent link must be read from the robot model it is attached to. -->
+      <parent link="tool0"/>
+      <child link="${prefix}onrobot_vgc10_base_link"/>
+      <!-- The tool is directly attached to the flange. -->
+      <origin rpy="0 0 0" xyz="0 0 0"/>
+    </joint>
+  </xacro:macro>
+  <xacro:macro name="finger_links" params="prefix">
+    <xacro:suction prefix="${prefix}"/>
+  </xacro:macro>
+  <xacro:macro name="suction" params="prefix">
+    <link name="${prefix}suction">
+      <inertial>
+        <origin xyz="0.0 0.0 0.0" rpy="0 0 0" />
+        <mass value="0.2" />
+        <inertia ixx="1.0E-03" ixy="1.0E-06" ixz="1.0E-06" iyy="1.0E-03" iyz="1.0E-06" izz="1.0E-03" />
+      </inertial>
+      <visual>
+        <origin xyz="0 0 0" rpy="0 0 0" />
+        <geometry>
+          <mesh filename="package://vgc10_description/meshes/visual/suction_cup.stl" />
+        </geometry>
+        <material name="">
+          <color rgba="0.9 0.9 0.9 1" />
+        </material>
+      </visual>
+      <collision>
+        <origin xyz="0 0 0" rpy="0 0 0" />
+        <geometry>
+          <mesh filename="package://vgc10_description/meshes/collision/suction_cup.stl" />
+        </geometry>
+      </collision>
+    </link>
+  </xacro:macro>
+  <xacro:macro name="suction_joint" params="prefix">
+    <joint name="${prefix}_suction_joint" type="fixed">
+      <origin xyz="0 0 0.094901" rpy="0 0 0" />
+      <parent link="${prefix}onrobot_vgc10_base_link" />
+      <child link="${prefix}suction" />
+      <axis xyz="1 0 0" />
+    </joint>
+  </xacro:macro>
+  <xacro:macro name="onrobot_vgc10" params="prefix">
+    <xacro:onrobot_vgc10_base_link prefix="${prefix}"/>
+    <xacro:finger_links prefix="${prefix}"/>
+    <xacro:suction_joint prefix="${prefix}"/>
+  </xacro:macro>
+   <!-- parameters -->
+   <xacro:arg name="prefix" default="" />
+   <xacro:arg name="joint_limit_params" default=""/>
+   <xacro:arg name="kinematics_params" default=""/>
+   <xacro:arg name="physical_params" default=""/>
+   <xacro:arg name="visual_params" default=""/>
+   <xacro:arg name="transmission_hw_interface" default=""/>
+   <xacro:arg name="safety_limits" default="false"/>
+   <xacro:arg name="safety_pos_margin" default="0.15"/>
+   <xacro:arg name="safety_k_position" default="20"/>
+   <!-- ros2_control related parameters -->
+   <xacro:arg name="use_fake_hardware" default="false" />
+   <xacro:arg name="fake_sensor_commands" default="false" />
+   <!-- ************************************************************************* -->
+   <!-- UR macro -->
   <xacro:include filename="$(find vgc10_description)/urdf/inc/ur_transmissions.xacro" />
   <xacro:include filename="$(find vgc10_description)/urdf/inc/ur_common.xacro" />
@@ -55,6 +106,5 @@
     safety_k_position:=20
     use_fake_hardware:=false
-    fake_sensor_commands:=false
-    initial_positions:=${dict(shoulder_pan_joint=0.0,shoulder_lift_joint=-1.57,elbow_joint=0.0,wrist_1_joint=-1.57,wrist_2_joint=0.0,wrist_3_joint=0.0)}">
+    fake_sensor_commands:=false">
     <!-- Load configuration data from the provided .yaml files -->
     <xacro:read_model_data
@@ -69,10 +119,211 @@
     <xacro:arg name="robot_ip" default="10.0.1.186"/>
     <!-- ros2 control include -->
-    <xacro:include filename="$(find vgc10_description)/urdf/ur.ros2_control.xacro" />
+    <!-- ********************************************************************************************** -->
+    <!-- ros2 control macro -->
+    <xacro:macro name="ur_ros2_control" params="name prefix
+      use_fake_hardware:=false fake_sensor_commands:=false
+      script_filename output_recipe_filename
+      input_recipe_filename tf_prefix
+      hash_kinematics robot_ip">
+      <ros2_control name="${name}" type="system">
+        <hardware>
+            <plugin>webots_ros2_control::Ros2ControlSystem</plugin>
+        </hardware>
+        <joint name="${prefix}shoulder_pan_joint">
+          <command_interface name="position">
+            <param name="min">${-2*pi}</param>
+            <param name="max">${2*pi}</param>
+          </command_interface>
+          <command_interface name="velocity">
+            <param name="min">-3.15</param>
+            <param name="max">3.15</param>
+          </command_interface>
+          <state_interface name="position"/>
+          <state_interface name="velocity"/>
+          <state_interface name="effort"/>
+        </joint>
+        <joint name="${prefix}shoulder_lift_joint">
+          <command_interface name="position">
+            <param name="min">${-2*pi}</param>
+            <param name="max">${2*pi}</param>
+          </command_interface>
+          <command_interface name="velocity">
+            <param name="min">-3.15</param>
+            <param name="max">3.15</param>
+          </command_interface>
+          <state_interface name="position"/>
+          <state_interface name="velocity"/>
+          <state_interface name="effort"/>
+        </joint>
+        <joint name="${prefix}elbow_joint">
+          <command_interface name="position">
+            <param name="min">${-pi}</param>
+            <param name="max">${pi}</param>
+          </command_interface>
+          <command_interface name="velocity">
+            <param name="min">-3.15</param>
+            <param name="max">3.15</param>
+          </command_interface>
+          <state_interface name="position"/>
+          <state_interface name="velocity"/>
+          <state_interface name="effort"/>
+        </joint>
+        <joint name="${prefix}wrist_1_joint">
+          <command_interface name="position">
+            <param name="min">${-2*pi}</param>
+            <param name="max">${2*pi}</param>
+          </command_interface>
+          <command_interface name="velocity">
+            <param name="min">-3.2</param>
+            <param name="max">3.2</param>
+          </command_interface>
+          <state_interface name="position"/>
+          <state_interface name="velocity"/>
+          <state_interface name="effort"/>
+        </joint>
+        <joint name="${prefix}wrist_2_joint">
+          <command_interface name="position">
+            <param name="min">${-2*pi}</param>
+            <param name="max">${2*pi}</param>
+          </command_interface>
+          <command_interface name="velocity">
+            <param name="min">-3.2</param>
+            <param name="max">3.2</param>
+          </command_interface>
+          <state_interface name="position"/>
+          <state_interface name="velocity"/>
+          <state_interface name="effort"/>
+        </joint>
+        <joint name="${prefix}wrist_3_joint">
+          <command_interface name="position">
+            <param name="min">${-2*pi}</param>
+            <param name="max">${2*pi}</param>
+          </command_interface>
+          <command_interface name="velocity">
+            <param name="min">-3.2</param>
+            <param name="max">3.2</param>
+          </command_interface>
+          <state_interface name="position"/>
+          <state_interface name="velocity"/>
+          <state_interface name="effort"/>
+        </joint>
+        <sensor name="tcp_fts_sensor">
+          <state_interface name="force.x"/>
+          <state_interface name="force.y"/>
+          <state_interface name="force.z"/>
+          <state_interface name="torque.x"/>
+          <state_interface name="torque.y"/>
+          <state_interface name="torque.z"/>
+        </sensor>
+        <!-- NOTE The following are joints used only for testing with fake hardware and will change in the future -->
+        <joint name="speed_scaling">
+          <state_interface name="speed_scaling_factor"/>
+          <param name="initial_speed_scaling_factor">1</param>
+          <command_interface name="target_speed_fraction_cmd"/>
+          <command_interface name="target_speed_fraction_async_success"/>
+        </joint>
+        <joint name="gpio">
+          <command_interface name="standard_digital_output_cmd_0"/>
+          <command_interface name="standard_digital_output_cmd_1"/>
+          <command_interface name="standard_digital_output_cmd_2"/>
+          <command_interface name="standard_digital_output_cmd_3"/>
+          <command_interface name="standard_digital_output_cmd_4"/>
+          <command_interface name="standard_digital_output_cmd_5"/>
+          <command_interface name="standard_digital_output_cmd_6"/>
+          <command_interface name="standard_digital_output_cmd_7"/>
+          <command_interface name="standard_digital_output_cmd_8"/>
+          <command_interface name="standard_digital_output_cmd_9"/>
+          <command_interface name="standard_digital_output_cmd_10"/>
+          <command_interface name="standard_digital_output_cmd_11"/>
+          <command_interface name="standard_digital_output_cmd_12"/>
+          <command_interface name="standard_digital_output_cmd_13"/>
+          <command_interface name="standard_digital_output_cmd_14"/>
+          <command_interface name="standard_digital_output_cmd_15"/>
+          <command_interface name="standard_digital_output_cmd_16"/>
+          <command_interface name="standard_digital_output_cmd_17"/>
+          <command_interface name="standard_analog_output_cmd_0"/>
+          <command_interface name="standard_analog_output_cmd_1"/>
+          <command_interface name="io_async_success"/>
+          <state_interface name="digital_output_0"/>
+          <state_interface name="digital_output_1"/>
+          <state_interface name="digital_output_2"/>
+          <state_interface name="digital_output_3"/>
+          <state_interface name="digital_output_4"/>
+          <state_interface name="digital_output_5"/>
+          <state_interface name="digital_output_6"/>
+          <state_interface name="digital_output_7"/>
+          <state_interface name="digital_output_8"/>
+          <state_interface name="digital_output_9"/>
+          <state_interface name="digital_output_10"/>
+          <state_interface name="digital_output_11"/>
+          <state_interface name="digital_output_12"/>
+          <state_interface name="digital_output_13"/>
+          <state_interface name="digital_output_14"/>
+          <state_interface name="digital_output_15"/>
+          <state_interface name="digital_output_16"/>
+          <state_interface name="digital_output_17"/>
+          <state_interface name="digital_input_0"/>
+          <state_interface name="digital_input_1"/>
+          <state_interface name="digital_input_2"/>
+          <state_interface name="digital_input_3"/>
+          <state_interface name="digital_input_4"/>
+          <state_interface name="digital_input_5"/>
+          <state_interface name="digital_input_6"/>
+          <state_interface name="digital_input_7"/>
+          <state_interface name="digital_input_8"/>
+          <state_interface name="digital_input_9"/>
+          <state_interface name="digital_input_10"/>
+          <state_interface name="digital_input_11"/>
+          <state_interface name="digital_input_12"/>
+          <state_interface name="digital_input_13"/>
+          <state_interface name="digital_input_14"/>
+          <state_interface name="digital_input_15"/>
+          <state_interface name="digital_input_16"/>
+          <state_interface name="digital_input_17"/>
+          <state_interface name="standard_analog_output_0"/>
+          <state_interface name="standard_analog_output_1"/>
+          <state_interface name="standard_analog_input_0"/>
+          <state_interface name="standard_analog_input_1"/>
+          <state_interface name="analog_io_type_0"/>
+          <state_interface name="analog_io_type_1"/>
+          <state_interface name="analog_io_type_2"/>
+          <state_interface name="analog_io_type_3"/>
+          <state_interface name="tool_mode"/>
+          <state_interface name="tool_output_voltage"/>
+          <state_interface name="tool_output_current"/>
+          <state_interface name="tool_temperature"/>
+          <state_interface name="tool_analog_input_0"/>
+          <state_interface name="tool_analog_input_1"/>
+          <state_interface name="tool_analog_input_type_0"/>
+          <state_interface name="tool_analog_input_type_1"/>
+          <state_interface name="robot_mode"/>
+          <state_interface name="robot_status_bit_0"/>
+          <state_interface name="robot_status_bit_1"/>
+          <state_interface name="robot_status_bit_2"/>
+          <state_interface name="robot_status_bit_3"/>
+          <state_interface name="safety_mode"/>
+          <state_interface name="safety_status_bit_0"/>
+          <state_interface name="safety_status_bit_1"/>
+          <state_interface name="safety_status_bit_2"/>
+          <state_interface name="safety_status_bit_3"/>
+          <state_interface name="safety_status_bit_4"/>
+          <state_interface name="safety_status_bit_5"/>
+          <state_interface name="safety_status_bit_6"/>
+          <state_interface name="safety_status_bit_7"/>
+          <state_interface name="safety_status_bit_8"/>
+          <state_interface name="safety_status_bit_9"/>
+          <state_interface name="safety_status_bit_10"/>
+          <state_interface name="program_running"/>
+        </joint>
+        <gpio name="system_interface">
+          <state_interface name="initialized"/>
+        </gpio>
+      </ros2_control>
+    </xacro:macro>
+    <!-- ********************************************************************************************** -->
     <!-- ros2 control instance -->
     <xacro:ur_ros2_control
       name="URPositionHardwareInterface" prefix="${prefix}"
       use_fake_hardware="$(arg use_fake_hardware)"
-      initial_positions="${initial_positions}"
       fake_sensor_commands="$(arg fake_sensor_commands)"
       script_filename="$(arg script_filename)"
@@ -382,3 +633,18 @@
     </joint>
   </xacro:macro>
+   <!-- ************************************************************************* -->
+   <!-- arm -->
+   <xacro:ur_robot
+     prefix="$(arg prefix)"
+     joint_limits_parameters_file="$(arg joint_limit_params)"
+     kinematics_parameters_file="$(arg kinematics_params)"
+     physical_parameters_file="$(arg physical_params)"
+     visual_parameters_file="$(arg visual_params)"
+     transmission_hw_interface="$(arg transmission_hw_interface)"
+     safety_limits="$(arg safety_limits)"
+     safety_pos_margin="$(arg safety_pos_margin)"
+     safety_k_position="$(arg safety_k_position)"
+     use_fake_hardware="$(arg use_fake_hardware)"
+     fake_sensor_commands="$(arg fake_sensor_commands)"/>
+  <xacro:onrobot_vgc10 prefix=""/>
 </robot>
